Commit message: convert several joints and links from sdf format to urdf format; tested

File: panda_description/xacro/macro.panda.urdf.xacro (robot description, xacro)
@@ -287,28 +287,20 @@
             <dynamics damping="0.3" />
         </joint>
+        <link name="rgbd_camera_link">
+            <origin xyz="0 0 0" rpy="0 0 0" />
+        </link>
         <joint name="panda_camera_joint" type="fixed">
-        <pose relative_to="panda_link7">0.01 0 0.01 0 0 0</pose>
-        <parent>panda_link7</parent>
-        <child>rgbd_camera_link</child>
-        </joint>
-        <link name="rgbd_camera_link">
-        <pose relative_to="panda_camera_joint">0 0 0 0 0 0</pose>
-        </link>
-        <joint name="panda_joint8" type="fixed">
-        <pose relative_to="panda_link7">0 0 0.107 0 0 0</pose>
-        <parent>panda_link7</parent>
-        <child>panda_link8</child>
-        </joint>
-        <link name='panda_link8'>
-        <pose relative_to="panda_joint8">0 0 0 0 0 0</pose>
+            <origin xyz="0.1 0 0.1" rpy="0 0 0" />
+            <parent link="panda_link7" />
+            <child link="rgbd_camera_link" />
+        </joint>
+        <link name='panda_tcp'>
+            <origin xyz="0 0 0" rpy="0 0 0" />
         </link>
         <joint name="panda_joint10" type="fixed">
-        <pose relative_to="panda_hand">0 0 0.100 0 0 0</pose>
-        <parent>panda_hand</parent>
-        <child>panda_tcp</child>
-        </joint>
-        <link name='panda_tcp'>
-        <pose relative_to="panda_joint10">0 0 0 0 0 0</pose>
-        </link>
+            <origin rpy="0 0 0" xyz="0 0 0.100" />
+            <parent link="panda_hand" />
+            <child link="panda_tcp" />
+        </joint>
     </xacro:macro>
 </robot>

Commit message: add fixed world link and joint for testing, has some conflictions with gazebo world link that need testing, needs to be argument based link for more modularity

File: panda_description/xacro/macro.panda.urdf.xacro (robot description, xacro)
@@ -6,4 +6,9 @@
 <!-- =================================================================================== -->
     <xacro:macro name="panda" params="ns prefix" >
+        <!-- <link name="world" />
+        <joint name="world_joint" type="fixed">
+            <parent link="world" />
+            <child link="panda_link0" />
+        </joint> -->
         <link name="panda_link0">
             <visual>

Commit message: add in joint with  parent link tag to allow modular robot placement within simulation world or model placement for rviz

File: panda_description/xacro/macro.panda.urdf.xacro (robot description, xacro)
@@ -5,10 +5,5 @@
 <!-- |    EDITING THIS FILE BY HAND IS NOT RECOMMENDED                                 | -->
 <!-- =================================================================================== -->
-    <xacro:macro name="panda" params="ns prefix" >
-        <!-- <link name="world" />
-        <joint name="world_joint" type="fixed">
-            <parent link="world" />
-            <child link="panda_link0" />
-        </joint> -->
+    <xacro:macro name="panda" params="ns prefix parent" >
         <link name="panda_link0">
             <visual>
@@ -28,4 +23,9 @@
             </inertial>
         </link>
+        <joint name="panda_joint0" type="fixed">
+            <origin rpy="0 0 0" xyz="0 0 0.25"/>
+            <parent link="${parent}"/>
+            <child link="panda_link0"/>
+        </joint>
         <link name="panda_link1">
             <visual>
