Commit message: add in example pedestal unit and parent argument for robot urdf.xacro for demonstration, TODO: extrapolate into separate .xacro file for table and pedestal for simulation

File: panda_description/xacro/panda.urdf.xacro (robot description, xacro)
@@ -16,4 +16,29 @@
   <xacro:panda_ros2_control ns="$(arg ns)" prefix="$(arg prefix)" />
   <!-- Arm -->
-  <xacro:panda ns="$(arg ns)" prefix="$(arg prefix)" />
+  <xacro:panda ns="$(arg ns)" prefix="$(arg prefix)" parent="mounting_block" />
+  <!-- World link inclusion -->
+  <!-- <link name="world" /> -->
+  <!-- Create a very heavy, inert base to be used as a mounting point for the arm-->
+  <link name="mounting_block">
+    <visual>
+      <origin xyz="0 0 0" rpy="0 0 0" />
+      <geometry>
+        <box size="0.5 0.5 0.5" />
+      </geometry>
+      <material name="gray">
+        <color rgba="0.4 0.4 0.4 1.0"/>
+      </material>
+    </visual>
+    <collision>
+      <origin xyz="0 0 0" rpy="0 0 0" />
+      <geometry>
+        <box size="0.5 0.5 0.5" />
+      </geometry>
+    </collision>
+    <inertial>
+      <origin xyz="0 0 0" rpy="0 0 0" />
+      <mass value="500.0"/> <!-- very heavy block -->
+      <inertia ixx="10.0" iyy="10.0" izz="10.0" ixy="0.0" ixz="0.0" iyz="0.0"/>
+    </inertial>
+  </link>
 </robot>

Commit message: remove commented world link line, better practice to add an object to attach robot model to

File: panda_description/xacro/panda.urdf.xacro (robot description, xacro)
@@ -17,6 +17,4 @@
   <!-- Arm -->
   <xacro:panda ns="$(arg ns)" prefix="$(arg prefix)" parent="mounting_block" />
-  <!-- World link inclusion -->
-  <!-- <link name="world" /> -->
   <!-- Create a very heavy, inert base to be used as a mounting point for the arm-->
   <link name="mounting_block">
