Commit message: removed double transmission tag; had two transmissions for joint 7

File: panda_description/xacro/macro.transmission.xacro (robot description, xacro)
@@ -65,13 +65,4 @@
       </actuator>
     </transmission>
-    <transmission name="${prefix}trans_7">
-      <type>transmission_interface/TransmissionInterface</type>
-      <joint name="${prefix}panda_finger_joint1">
-        <hardwareInterface>${hw_iface}</hardwareInterface>
-      </joint>
-      <actuator name="${prefix}motor_7">
-        <mechanicalReduction>1</mechanicalReduction>
-      </actuator>
-    </transmission>
   </xacro:macro>
 </robot>

Commit message: add tag for finger joint back in, accidentally removed

File: panda_description/xacro/macro.transmission.xacro (robot description, xacro)
@@ -65,4 +65,13 @@
       </actuator>
     </transmission>
+    <transmission name="${prefix}trans_7">
+      <type>transmission_interface/TransmissionInterface</type>
+      <joint name="${prefix}panda_finger_joint1">
+        <hardwareInterface>${hw_iface}</hardwareInterface>
+      </joint>
+      <actuator name="${prefix}motor_7">
+        <mechanicalReduction>1</mechanicalReduction>
+      </actuator>
+    </transmission>
   </xacro:macro>
 </robot>
